File: compute_module.kicad_pcb (KiCad board)
At the start: 4 copper layers, 93.2 x 62.4 mm, 66 parts, among them J1 2001-1-2-21-00-BK, J2 JC-128, P1 POWER, P2 HOST, P3 CAM1, P4 CONN_02X20, Q1 2N7002P.215, Q2 DMP3056L-7, Q3 2N7002P.215, U1 REG1117-3.3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

Commit message: pcb: angelinux board respin
This patch changes the board sinkscreen to Angelinux
Other:
- board text added: "ANGELINUX Rpi Module Base Board Rev: A"
- board text removed: "Compute Module Base Board Rev: A"
Changed lines of the file:
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@@
-(kicad_pcb (version 4) (host pcbnew 4.0.5+dfsg1-4)
+(kicad_pcb (version 20171130) (host pcbnew 5.1.2-f72e74a~84~ubuntu16.04.1)
   (general
-    (links 282)
-    (no_connects 0)
-    (area 87.524999 43.924999 180.875001 106.475001)
     (thickness 1.6)
     (drawings 14)
@@
   (page A4)
   (layers
-    (0 F.Cu signal)
-    (1 In1.Cu power)
-    (2 In2.Cu mixed)
-    (31 B.Cu signal)
-    (32 B.Adhes user)
-    (33 F.Adhes user)
-    (34 B.Paste user)
-    (35 F.Paste user)
+    (0 F.Cu signal hide)
+    (1 In1.Cu power hide)
+    (2 In2.Cu mixed hide)
+    (31 B.Cu signal hide)
+    (32 B.Adhes user hide)
+    (33 F.Adhes user hide)
+    (34 B.Paste user hide)
+    (35 F.Paste user hide)
     (36 B.SilkS user)
     (37 F.SilkS user)
     (38 B.Mask user)
     (39 F.Mask user)
-    (40 Dwgs.User user)
-    (41 Cmts.User user)
-    (42 Eco1.User user)
-    (43 Eco2.User user)
-    (44 Edge.Cuts user)
-    (45 Margin user)
-    (46 B.CrtYd user)
-    (47 F.CrtYd user)
-    (48 B.Fab user)
-    (49 F.Fab user)
+    (40 Dwgs.User user hide)
+    (41 Cmts.User user hide)
+    (42 Eco1.User user hide)
+    (43 Eco2.User user hide)
+    (44 Edge.Cuts user hide)
+    (45 Margin user hide)
+    (46 B.CrtYd user hide)
+    (47 F.CrtYd user hide)
+    (48 B.Fab user hide)
+    (49 F.Fab user hide)
   )
   (setup
@@
     (zone_45_only no)
     (trace_min 0.2)
-    (segment_width 0.2)
-    (edge_width 0.15)
     (via_size 0.45)
     (via_drill 0.3)
@@
     (uvia_min_size 0.2)
     (uvia_min_drill 0.1)
+    (edge_width 0.15)
+    (segment_width 0.2)
     (pcb_text_width 0.3)
     (pcb_text_size 1.5 1.5)
@@
     (visible_elements FFFFFF7F)
     (pcbplotparams
-      (layerselection 0x00030_80000001)
+      (layerselection 0x010f0_ffffffff)
       (usegerberextensions false)
+      (usegerberattributes false)
+      (usegerberadvancedattributes false)
+      (creategerberjobfile false)
       (excludeedgelayer true)
       (linewidth 0.100000)
@@
       (hpglpennumber 1)
       (hpglpenspeed 20)
-      (hpglpendiameter 15)
-      (hpglpenoverlay 2)
+      (hpglpendiameter 15.000000)
       (psnegative false)
       (psa4output false)
@@
       (outputformat 1)
       (mirror false)
-      (drillshape 1)
+      (drillshape 0)
       (scaleselection 1)
-      (outputdirectory ""))
+      (outputdirectory "angelinux/"))
   )
   (net 0 "")
@@
     (tags SOT-23)
     (attr smd)
-    (fp_text reference D3 (at 0.5 -3 360) (layer B.SilkS)
+    (fp_text reference D3 (at 0.5 -3) (layer B.SilkS)
       (effects (font (size 1 1) (thickness 0.15)) (justify mirror))
     )
@@
       (effects (font (size 1 1) (thickness 0.15)) (justify mirror))
     )
-    (fp_text user %R (at 0 0 360) (layer B.Fab)
+    (fp_text user %R (at 0 0) (layer B.Fab)
       (effects (font (size 0.5 0.5) (thickness 0.075)) (justify mirror))
     )
@@
       (effects (font (size 1 1) (thickness 0.15)) (justify mirror))
     )
-    (fp_text user %R (at 0 0 450) (layer B.Fab)
+    (fp_text user %R (at 0 0 90) (layer B.Fab)
       (effects (font (size 0.5 0.5) (thickness 0.075)) (justify mirror))
     )
@@
       (net 2 GND))
     (model ${KISYS3DMOD}/Connectors.3dshapes/USB_A.wrl
-      (at (xyz 0.14 0 0))
+      (offset (xyz 3.555999946594238 0 0))
       (scale (xyz 1 1 1))
       (rotate (xyz 0 0 90))
@@
     (tags SOT-23)
     (attr smd)
-    (fp_text reference Q1 (at 0 2.8 360) (layer F.SilkS)
+    (fp_text reference Q1 (at 0 2.8) (layer F.SilkS)
       (effects (font (size 1 1) (thickness 0.15)))
     )
@@
       (effects (font (size 1 1) (thickness 0.15)))
     )
-    (fp_text user %R (at 0 0 360) (layer F.Fab)
+    (fp_text user %R (at 0 0) (layer F.Fab)
       (effects (font (size 0.5 0.5) (thickness 0.075)))
     )
@@
     (tags "Fuse Sicherung SMD1206 Littlefuse-Wickmann Reflow ")
     (attr smd)
-    (fp_text reference F1 (at -2.6 0 360) (layer F.SilkS)
+    (fp_text reference F1 (at -2.6 0) (layer F.SilkS)
       (effects (font (size 1 1) (thickness 0.15)))
     )
@@
       (net 130 GPIO21))
     (model Pin_Headers.3dshapes/Pin_Header_Straight_2x20.wrl
-      (at (xyz 0.05 -0.95 0))
+      (offset (xyz 1.269999980926514 -24.12999963760376 0))
       (scale (xyz 1 1 1))
       (rotate (xyz 0 0 90))
@@
     (tags SOT-23)
     (attr smd)
-    (fp_text reference D9 (at -2.4 0 360) (layer F.SilkS)
+    (fp_text reference D9 (at -2.4 0) (layer F.SilkS)
       (effects (font (size 1 1) (thickness 0.15)))
     )
@@
       (effects (font (size 1 1) (thickness 0.15)))
     )
-    (fp_text user %R (at 0 0 360) (layer F.Fab)
+    (fp_text user %R (at 0 0) (layer F.Fab)
       (effects (font (size 0.5 0.5) (thickness 0.075)))
     )
@@
     (tags SOT-23)
     (attr smd)
-    (fp_text reference D10 (at -2.4 0 360) (layer F.SilkS)
+    (fp_text reference D10 (at -2.4 0) (layer F.SilkS)
       (effects (font (size 1 1) (thickness 0.15)))
     )
@@
       (effects (font (size 1 1) (thickness 0.15)))
     )
-    (fp_text user %R (at 0 0 360) (layer F.Fab)
+    (fp_text user %R (at 0 0) (layer F.Fab)
       (effects (font (size 0.5 0.5) (thickness 0.075)))
     )
@@
     (effects (font (size 1 1) (thickness 0.15)))
   )
-  (gr_text "Compute Module Base Board\nRev: A" (at 92.2 53.4) (layer F.SilkS)
+  (gr_text "ANGELINUX Rpi Module Base Board\nRev: A" (at 92.2 53.4) (layer F.SilkS)
     (effects (font (size 1.4 1.4) (thickness 0.25)) (justify left))
   )
